File: RF/OPA2000_RF/RF_output/RF_output.kicad_pcb (KiCad board)
At the start: 2 copper layers, 100 x 100 mm, 36 parts, among them J1 Conn_Coaxial, J2 VDD in, J3 GND, Q1 BLF188XR

Commit message: MCU2 sch done
Parts:
- removed 1:9 Transformer: Laird_28B1020_100, MyPCBLib:Laird_28B1020_100 (x2)
- removed BALUN: Laird_28B1020_100, MyPCBLib:Laird_28B1020_100
- removed C15, C5, C6, C7, C8: 103, Capacitors_SMD:C_1206_HandSoldering
- removed DC Feed: Laird_28B1020_100, MyPCBLib:Laird_28B1020_100
- removed J1: Conn_Coaxial, MyPCBLib:RF_conn_pad
- removed SC6: GND, MyPCBLib:M3_Screwhole
- removed SYM1: Symbol_HighVoltage_Type2_SilkTop_VerySmall, MyPCBLib:Symbol_HighVoltage_Type2_SilkTop_VerySmall
- added C23: 30pF, Capacitor_SMD:C_1210_3225Metric_Pad1.33x2.70mm_HandSolder, F.Cu at (137.2, 62.8)
- added C24: 103, Capacitor_SMD:C_1206_3216Metric_Pad1.33x1.80mm_HandSolder, F.Cu at (134.8, 130.2)
- added C25: 103, Capacitor_SMD:C_1206_3216Metric_Pad1.33x1.80mm_HandSolder, F.Cu at (132.0, 130.2)
- added C26: 103, Capacitor_SMD:C_1206_3216Metric_Pad1.33x1.80mm_HandSolder, F.Cu at (129.2, 130.2)
- added C27: 103, Capacitor_SMD:C_1206_3216Metric_Pad1.33x1.80mm_HandSolder, F.Cu at (134.5, 70.8)
- added C28: 103, Capacitor_SMD:C_1206_3216Metric_Pad1.33x1.80mm_HandSolder, F.Cu at (131.5, 70.8)
- added C29: 103, Capacitor_SMD:C_1206_3216Metric_Pad1.33x1.80mm_HandSolder, F.Cu at (128.5, 70.8)
- added C30: 220uF 100V, Capacitor_SMD:CP_Elec_10x10.5, F.Cu at (142.8, 126.2)
- added C31: 220uF 100V, Capacitor_SMD:CP_Elec_10x10.5, F.Cu at (142.5, 75.0)
- added F1: 30A, MyPCBLib:Fuseholder_Littelfuse_Nano2_456, F.Cu at (141.5, 116.0)
- added F2: 30A, MyPCBLib:Fuseholder_Littelfuse_Nano2_456, F.Cu at (141.5, 85.8)
- added L1: Choke, MyPCBLib:5943004901, F.Cu at (78.8, 88.8)
- added L2: Choke, MyPCBLib:5943004901, F.Cu at (78.8, 111.5)
- added Q2: BLF188XR, MyPCBLib:BLF188XR, F.Cu at (44.0, 123.5)
- added T1: TLT, MyPCBLib:Laird_28B1020_100, F.Cu at (73.2, 66.0)
- added T2: TLT, MyPCBLib:Laird_28B1020_100, F.Cu at (73.2, 134.5)
- added T3: TLT, MyPCBLib:Laird_28B1020_100, F.Cu at (110.0, 66.0)
- added T4: TLT, MyPCBLib:Laird_28B1020_100, F.Cu at (109.5, 134.5)
- added T5: TLT, MyPCBLib:Laird_28B1020_100, F.Cu at (115.2, 100.0)
- added e1: Conn_Coaxial, MyPCBLib:RF_conn_pad_short, F.Cu at (145.0, 59.8)
- C1, C2, C3, C4: footprint Capacitors_SMD:C_1210_HandSoldering -> Capacitor_SMD:C_1210_3225Metric_Pad1.33x2.70mm_HandSolder
- C10, C9: value 220uF 100V -> 103; footprint Capacitors_SMD:CP_Elec_10x10.5 -> Capacitor_SMD:C_1206_3216Metric_Pad1.33x1.80mm_HandSolder
- C11, C12, C13, C14, C16, C17, C18, C19, C20: footprint Capacitors_SMD:C_1206_HandSoldering -> Capacitor_SMD:C_1206_3216Metric_Pad1.33x1.80mm_HandSolder
- C21: value 30pF -> 103; footprint Capacitors_SMD:C_1210_HandSoldering -> Capacitor_SMD:C_1206_3216Metric_Pad1.33x1.80mm_HandSolder
- J2: value VDD in -> GND
- J3: value GND -> VDD in
- moved SC1 65.2 mm to (55.0, 145.0)
- moved J2 41.8 mm to (138.8, 140.8), turned to 180 degrees
- moved J3 34.1 mm to (143.0, 100.0)
- moved C9 28.9 mm to (119.2, 95.5)
- moved C21 27.9 mm to (119.3, 117.8), turned to 0 degrees
- moved Q1 23.5 mm to (44.0, 76.5)
- moved C14 23.3 mm to (119.2, 83.0)
- moved C13 21.3 mm to (119.2, 85.5)
- moved C10 21.2 mm to (119.2, 93.0)
- moved SC3 20.9 mm to (54.0, 100.0)
- moved C11 20.5 mm to (119.2, 90.5)
- moved C20 20.4 mm to (119.3, 115.2)
- moved C17 20.4 mm to (119.2, 107.8)
- moved C18 20.4 mm to (119.2, 110.2)
- moved C19 20.4 mm to (119.2, 112.8)
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Connections:
- C1 pad 1: D1 -> Net-(C1-Pad1)
- C10 pad 1: VDD -> Net-(C10-Pad1)
- C10 pad 2: GNDPWR -> Net-(C10-Pad2)
- C11 pad 1: Net-(C11-Pad1) -> Net-(C10-Pad1)
- C11 pad 2: Net-(C11-Pad2) -> Net-(C10-Pad2)
- C12 pad 1: Net-(C11-Pad1) -> Net-(C10-Pad1)
- C12 pad 2: Net-(C11-Pad2) -> Net-(C10-Pad2)
- C13 pad 1: Net-(C11-Pad1) -> Net-(C10-Pad1)
- C13 pad 2: Net-(C11-Pad2) -> Net-(C10-Pad2)
- C14 pad 1: Net-(C11-Pad1) -> Net-(C10-Pad1)
- C14 pad 2: Net-(C11-Pad2) -> Net-(C10-Pad2)
- C2 pad 1: D2 -> Net-(C2-Pad1)
- C21 pad 1: Net-(C21-Pad1) -> Net-(C16-Pad1)
- C21 pad 2: GNDPWR -> Net-(C16-Pad2)
- C3 pad 1: D1 -> Net-(C1-Pad1)
- C4 pad 1: D2 -> Net-(C2-Pad1)
- C9 pad 1: VDD -> Net-(C10-Pad1)
- C9 pad 2: GNDPWR -> Net-(C10-Pad2)
- J2 pad 1: VDD -> GNDPWR
- J3 pad 1: GNDPWR -> VDD
- Q1 pad 1: D1 -> Net-(C1-Pad1)
- Q1 pad 2: D2 -> Net-(C1-Pad1)
Routing:
- net GNDPWR: track 0.00 -> 24.0 mm, vias 512 -> 419
- net (no net): vias 0 -> 1
- added copper zone on F.Cu, net (none)
- added copper zone on F.Cu, net Net-(C1-Pad1)
- added copper zone on F.Cu, net Net-(C10-Pad1)
- added copper zone on F.Cu, net Net-(C10-Pad2)
- added copper zone on F.Cu, net Net-(C2-Pad1)
- added copper zone on F.Cu, net Net-(C24-Pad2)
- added copper zone on F.Cu, net Net-(C27-Pad2)
- removed copper zone on F.Cu, net D1
- removed copper zone on F.Cu, net D2
- removed copper zone on F.Cu, net Net-(C11-Pad1)
- removed copper zone on F.Cu, net Net-(C11-Pad2)
Other:
- board text added: "OPA2000 DUAL LDMOS OUTPUT V0.1"
- board text added: "Zening Lu (BI4WOP) July 17, 2021 Visit www.zening.lu for more Info"
- board text removed: "Caution: RF Electric Shock"
- board text removed: "D1"
- board text removed: "D2"
- board text removed: "GND"
- board text removed: "OPA1000 Solid State Power Amplifier RF Output Board V0.1"
- board text removed: "Output"
- board text removed: "VDD +50V"
- board text removed: "Zening Lu (BI4WOP) Dec 10, 2019 Visit www.zening.lu for more information"
