File: MCU/MCU_2/OutputSignals.sch (KiCad schematic (older format))
At the start: 30 parts, among them J11 In Relay, J12 Out Relay, J13 ALC out, Q12 DTC144E, Q18 DTA144E, Q19 DTA144E, Q2 8050, Q3 8050, Q5 DTA144E, Q8 DTA144E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

Commit message: routing signals
Parts:
- added C47, C5, C69: 104, lc_lib:0805_C, symbol Device:C_Small
- C35, C36: symbol Device:CP_Small -> Device:C_Small
- SW1: footprint lc_lib:DIP-8 -> Button_Switch_SMD:SW_DIP_SPSTx04_Slide_KingTek_DSHP04TS_W7.62mm_P1.27mm
Connections:
- net +3V3: now also C47.2, C69.2
- net GND: now also C47.1, C5.1, C69.1
- net at U8.5 (CV): now also C5.2
Changed lines of the file:
@@
 $Descr A4 11693 8268
 encoding utf-8
-Sheet 3 5
+Sheet 5 5
 Title ""
 Date ""
@@
 	3350 1700 3150 1700
 $Comp
-L Device:CP_Small C35
+L Device:C_Small C35
 U 1 1 5E7F3AB6
 P 3350 1500
@@
 $EndComp
 $Comp
-L Device:CP_Small C36
+L Device:C_Small C36
 U 1 1 5E7F8AB0
 P 3550 1500
@@
 $EndComp
 Wire Wire Line
-	5500 4400 5500 4500
+	5500 4400 5500 4450
 $Comp
 L Timer:TLC555xD U8
@@
 F 0 "SW1" V 3950 5500 50  0000 L CNN
 F 1 "SW_DIP_x04" V 4050 5500 50  0000 L CNN
-F 2 "lc_lib:DIP-8" H 3800 6050 50  0001 C CNN
+F 2 "Button_Switch_SMD:SW_DIP_SPSTx04_Slide_KingTek_DSHP04TS_W7.62mm_P1.27mm" H 3800 6050 50  0001 C CNN
 F 3 "~" H 3800 6050 50  0001 C CNN
 	1    3800 6050
@@
 Wire Wire Line
 	2950 2450 3100 2450
+$Comp
+L Device:C_Small C47
+U 1 1 620F1C78
+P 2050 1250
+F 0 "C47" H 1850 1350 50  0000 L CNN
+F 1 "104" H 1750 1200 50  0000 L CNN
+F 2 "lc_lib:0805_C" H 2050 1250 50  0001 C CNN
+F 3 "~" H 2050 1250 50  0001 C CNN
+	1    2050 1250
+	-1   0    0    1
+$EndComp
+Wire Wire Line
+	2050 1150 2050 1100
+Wire Wire Line
+	2050 1100 2250 1100
+Connection ~ 2250 1100
+Wire Wire Line
+	2050 1350 2050 1600
+Wire Wire Line
+	2050 1600 2200 1600
+Connection ~ 2200 1600
+$Comp
+L Device:C_Small C69
+U 1 1 620FCFA6
+P 5750 4450
+F 0 "C69" H 5550 4550 50  0000 L CNN
+F 1 "104" H 5450 4400 50  0000 L CNN
+F 2 "lc_lib:0805_C" H 5750 4450 50  0001 C CNN
+F 3 "~" H 5750 4450 50  0001 C CNN
+	1    5750 4450
+	0    1    1    0
+$EndComp
+Wire Wire Line
+	5650 4450 5500 4450
+Connection ~ 5500 4450
+Wire Wire Line
+	5500 4450 5500 4500
+$Comp
+L power:GND #PWR0118
+U 1 1 62101C97
+P 5950 4450
+F 0 "#PWR0118" H 5950 4200 50  0001 C CNN
+F 1 "GND" H 5955 4277 50  0000 C CNN
+F 2 "" H 5950 4450 50  0001 C CNN
+F 3 "" H 5950 4450 50  0001 C CNN
+	1    5950 4450
+	1    0    0    -1
+$EndComp
+Wire Wire Line
+	5950 4450 5850 4450
+$Comp
+L Device:C_Small C5
+U 1 1 6219A0D1
+P 4900 5250
+F 0 "C5" H 4700 5350 50  0000 L CNN
+F 1 "104" H 4600 5200 50  0000 L CNN
+F 2 "lc_lib:0805_C" H 4900 5250 50  0001 C CNN
+F 3 "~" H 4900 5250 50  0001 C CNN
+	1    4900 5250
+	-1   0    0    1
+$EndComp
+Wire Wire Line
+	4900 5150 4900 4900
+Wire Wire Line
+	4900 4900 5000 4900
+$Comp
+L power:GND #PWR0129
+U 1 1 6219F09B
+P 4900 5400
+F 0 "#PWR0129" H 4900 5150 50  0001 C CNN
+F 1 "GND" H 4905 5227 50  0000 C CNN
+F 2 "" H 4900 5400 50  0001 C CNN
+F 3 "" H 4900 5400 50  0001 C CNN
+	1    4900 5400
+	1    0    0    -1
+$EndComp
+Wire Wire Line
+	4900 5400 4900 5350
 $EndSCHEMATC
