File: MCU/MCU_2/MonitorInput.sch (KiCad schematic (older format))
At the start: 69 parts, among them J19 RF, J5 PowerSense, J6 NTC1, J7 NTC2, J8 SWR1, J9 SWR2, Q1 DTC144E, Q4 DTC144E, Q6 DTC144E, Q7 DTC144E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

Commit message: routing signals
Parts:
- C22, C23: value C_Small -> 104
Connections:
- net +5V: now also J8.1 (Pin_1), J9.1 (Pin_1); no longer J8.6 (Pin_6), J9.6 (Pin_6)
- net FWD1: now also J8.3 (Pin_3); no longer J8.4 (Pin_4)
- net FWD2: now also J9.3 (Pin_3); no longer J9.4 (Pin_4)
- net FWDpeak1: now also J8.2 (Pin_2); no longer J8.5 (Pin_5)
- net FWDpeak2: now also J9.2 (Pin_2); no longer J9.5 (Pin_5)
- net GNDA: now also J8.6 (Pin_6), J9.6 (Pin_6); no longer J8.1 (Pin_1), J9.1 (Pin_1)
- net REV1: now also J8.5 (Pin_5); no longer J8.2 (Pin_2)
- net REV2: now also J9.5 (Pin_5); no longer J9.2 (Pin_2)
- net REVpeak1: now also J8.4 (Pin_4); no longer J8.3 (Pin_3)
- net REVpeak2: now also J9.4 (Pin_4); no longer J9.3 (Pin_3)
Changed lines of the file:
@@
 L Connector_Generic:Conn_01x06 J8
 U 1 1 5E0EA526
-P 10550 3100
-F 0 "J8" H 10468 2575 50  0000 C CNN
-F 1 "SWR1" H 10468 2666 50  0000 C CNN
-F 2 "Connector_JST:JST_PH_B6B-PH-SM4-TB_1x06-1MP_P2.00mm_Vertical" H 10550 3100 50  0001 C CNN
-F 3 "~" H 10550 3100 50  0001 C CNN
-	1    10550 3100
-	1    0    0    1
+P 10550 3000
+F 0 "J8" H 10468 2475 50  0000 C CNN
+F 1 "SWR1" H 10468 2566 50  0000 C CNN
+F 2 "Connector_JST:JST_PH_B6B-PH-SM4-TB_1x06-1MP_P2.00mm_Vertical" H 10550 3000 50  0001 C CNN
+F 3 "~" H 10550 3000 50  0001 C CNN
+	1    10550 3000
+	1    0    0    -1
 $EndComp
 $Comp
 L Connector_Generic:Conn_01x06 J9
 U 1 1 5E0EBB82
-P 9700 3900
-F 0 "J9" H 9618 3375 50  0000 C CNN
-F 1 "SWR2" H 9618 3466 50  0000 C CNN
-F 2 "Connector_JST:JST_PH_B6B-PH-SM4-TB_1x06-1MP_P2.00mm_Vertical" H 9700 3900 50  0001 C CNN
-F 3 "~" H 9700 3900 50  0001 C CNN
-	1    9700 3900
-	1    0    0    1
+P 9700 3800
+F 0 "J9" H 9618 3275 50  0000 C CNN
+F 1 "SWR2" H 9618 3366 50  0000 C CNN
+F 2 "Connector_JST:JST_PH_B6B-PH-SM4-TB_1x06-1MP_P2.00mm_Vertical" H 9700 3800 50  0001 C CNN
+F 3 "~" H 9700 3800 50  0001 C CNN
+	1    9700 3800
+	1    0    0    -1
 $EndComp
 $Comp
@@
 	10250 3300 10350 3300
 Wire Wire Line
-	10150 2800 10350 2800
-Wire Wire Line
 	9000 3800 9500 3800
 Wire Wire Line
@@
 P 6050 950
 F 0 "C23" H 5750 1000 50  0000 L CNN
-F 1 "C_Small" H 5650 900 50  0000 L CNN
+F 1 "104" H 5650 900 50  0000 L CNN
 F 2 "lc_lib:0805_C" H 6050 950 50  0001 C CNN
 F 3 "~" H 6050 950 50  0001 C CNN
@@
 U 1 1 5E214358
 P 6100 4600
-F 0 "U6" H 6100 4967 50  0000 C CNN
-F 1 "LMV324" H 6100 4876 50  0000 C CNN
+F 0 "U6" H 5800 4950 50  0000 C CNN
+F 1 "LMV324" H 5750 4850 50  0000 C CNN
 F 2 "lc_lib:SOIC-14_150MIL" H 6050 4700 50  0001 C CNN
 F 3 "http://www.ti.com/lit/ds/symlink/lmv324.pdf" H 6150 4800 50  0001 C CNN
@@
 P 5900 4200
 F 0 "C22" H 5992 4246 50  0000 L CNN
-F 1 "C_Small" H 5992 4155 50  0000 L CNN
+F 1 "104" H 5992 4155 50  0000 L CNN
 F 2 "lc_lib:0805_C" H 5900 4200 50  0001 C CNN
 F 3 "~" H 5900 4200 50  0001 C CNN
@@
 P 2100 4550
 F 0 "U4" H 2250 4400 50  0000 C CNN
-F 1 "LMV324" H 2100 4826 50  0000 C CNN
+F 1 "LMV324" H 1550 4800 50  0000 C CNN
 F 2 "lc_lib:SOIC-14_150MIL" H 2050 4650 50  0001 C CNN
 F 3 "http://www.ti.com/lit/ds/symlink/lmv324.pdf" H 2150 4750 50  0001 C CNN
@@
 	1    0    0    -1
 $EndComp
-Wire Wire Line
-	10800 2800 10350 2800
-Connection ~ 10350 2800
 $Comp
 L power:GNDA #PWR0133
@@
 Text HLabel 2200 3550 0    50   Output ~ 0
 \Overdrive
+Wire Wire Line
+	10150 2800 10350 2800
+Connection ~ 10350 2800
+Wire Wire Line
+	10350 2800 10800 2800
 $EndSCHEMATC

Commit message: almost finished routing MCU2
Connections:
- net +5V renamed +5VA
Changed lines of the file:
@@
 Wire Wire Line
 	10150 2750 10150 2800
-$Comp
-L power:+5V #PWR064
-U 1 1 5E0F23A0
-P 10150 2750
-F 0 "#PWR064" H 10150 2600 50  0001 C CNN
-F 1 "+5V" H 10165 2923 50  0000 C CNN
-F 2 "" H 10150 2750 50  0001 C CNN
-F 3 "" H 10150 2750 50  0001 C CNN
-	1    10150 2750
-	1    0    0    -1
-$EndComp
 Wire Wire Line
 	9300 3600 9500 3600
-$Comp
-L power:+5V #PWR065
-U 1 1 5E0F465C
-P 9300 3600
-F 0 "#PWR065" H 9300 3450 50  0001 C CNN
-F 1 "+5V" H 9315 3773 50  0000 C CNN
-F 2 "" H 9300 3600 50  0001 C CNN
-F 3 "" H 9300 3600 50  0001 C CNN
-	1    9300 3600
-	1    0    0    -1
-$EndComp
 $Comp
 L power:GNDA #PWR038
@@
 Wire Wire Line
 	10350 2800 10800 2800
+$Comp
+L power:+5VA #PWR0132
+U 1 1 619316D6
+P 10150 2750
+F 0 "#PWR0132" H 10150 2600 50  0001 C CNN
+F 1 "+5VA" H 10165 2923 50  0000 C CNN
+F 2 "" H 10150 2750 50  0001 C CNN
+F 3 "" H 10150 2750 50  0001 C CNN
+	1    10150 2750
+	1    0    0    -1
+$EndComp
+$Comp
+L power:+5VA #PWR0158
+U 1 1 61931B01
+P 9300 3600
+F 0 "#PWR0158" H 9300 3450 50  0001 C CNN
+F 1 "+5VA" H 9315 3773 50  0000 C CNN
+F 2 "" H 9300 3600 50  0001 C CNN
+F 3 "" H 9300 3600 50  0001 C CNN
+	1    9300 3600
+	1    0    0    -1
+$EndComp
+Text GLabel 10550 4550 2    50   Output ~ 0
+PwrOnSig
+Wire Wire Line
+	10550 4550 10250 4550
+Text HLabel 10250 4550 0    50   Input ~ 0
+RF_bias_on
 $EndSCHEMATC
