File: MCU/MCU_2/Power.sch (KiCad schematic (older format))
At the start: 56 parts, among them J22 12Vin, J23 BIAS, M1 Fan, M2 Fan, Q10 AO3402, Q11 AO3402, Q16 2N5401, Q17 DTC144E, U10 MT2492/SY8120, U12 TL431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

Commit message: MCU PCB start layouting
Parts:
- removed C47: 104, lc_lib:0805_C, symbol Device:C_Small
- removed JP1: 0, lc_lib:0805_R, symbol Device:R_Small
- removed L4: BEAD, lc_lib:1206_L, symbol Device:L_Core_Ferrite
- added C68: 10uF, lc_lib:0805_C, symbol Device:C_Small
- C42: footprint Capacitor_THT:CP_Radial_D5.0mm_P2.50mm -> lc_lib:0805_C; symbol Device:CP_Small -> Device:C_Small
- C48: value 104 -> 10uF
- C63: value 10V 100uF -> 10uF; footprint Capacitor_THT:CP_Radial_D5.0mm_P2.50mm -> lc_lib:0805_C; symbol Device:CP_Small -> Device:C_Small
- L5: value 10uH -> 6.8uH
Connections:
- net +12V: now also C41.1, C42.1, R63.1, U10.5 (VIN)
- net +5VA: now also C68.1
- net GND: now also C68.2
Changed lines of the file:
@@
 P 3700 1650
 F 0 "L5" V 3925 1650 50  0000 C CNN
-F 1 "10uH" V 3834 1650 50  0000 C CNN
+F 1 "6.8uH" V 3834 1650 50  0000 C CNN
 F 2 "MyPCBLib:L_SMD4030_hand" H 3700 1650 50  0001 C CNN
 F 3 "~" H 3700 1650 50  0001 C CNN
@@
 	2100 1800 2100 1650
 $Comp
-L Device:CP_Small C42
+L Device:C_Small C42
 U 1 1 5F5CC649
 P 2100 1900
 F 0 "C42" H 2188 1946 50  0000 L CNN
 F 1 "10u" H 2188 1855 50  0000 L CNN
-F 2 "Capacitor_THT:CP_Radial_D5.0mm_P2.50mm" H 2100 1900 50  0001 C CNN
+F 2 "lc_lib:0805_C" H 2100 1900 50  0001 C CNN
 F 3 "~" H 2100 1900 50  0001 C CNN
 	1    2100 1900
@@
 Wire Wire Line
 	4700 2250 4700 2200
-$Comp
-L Device:C_Small C47
-U 1 1 5F5DD8A8
-P 5000 2000
-F 0 "C47" H 5100 2050 50  0000 L CNN
-F 1 "104" H 5100 1900 50  0000 L CNN
-F 2 "lc_lib:0805_C" H 5000 2000 50  0001 C CNN
-F 3 "~" H 5000 2000 50  0001 C CNN
-	1    5000 2000
-	1    0    0    -1
-$EndComp
-Wire Wire Line
-	5000 1900 5000 1650
-Wire Wire Line
-	5000 1650 4700 1650
 Connection ~ 4700 1650
-Wire Wire Line
-	5000 2100 5000 2200
-Wire Wire Line
-	5000 2200 4700 2200
 Connection ~ 4700 2200
 Wire Wire Line
@@
 	0    1    1    0
 $EndComp
-Connection ~ 5000 1650
 $Comp
 L Regulator_Linear:AZ1117-3.3 U13
@@
 	5750 3150 5750 3300
 Connection ~ 6250 2800
-Wire Wire Line
-	1200 1650 1400 1650
 $Comp
 L MySchLib:D_Zener D8
@@
 Wire Wire Line
 	1200 1800 1200 1750
-$Comp
-L Device:L_Core_Ferrite L4
-U 1 1 5E2A38D9
-P 1550 1650
-F 0 "L4" V 1775 1650 50  0000 C CNN
-F 1 "BEAD" V 1684 1650 50  0000 C CNN
-F 2 "lc_lib:1206_L" H 1550 1650 50  0001 C CNN
-F 3 "~" H 1550 1650 50  0001 C CNN
-	1    1550 1650
-	0    -1   -1   0
-$EndComp
-Wire Wire Line
-	5000 1650 5050 1650
 Connection ~ 5300 1650
 Wire Wire Line
-	5300 1650 5450 1650
+	5300 1650 5400 1650
 $Comp
 L Connector_Generic:Conn_01x01 SC1
@@
 	5800 4950 5800 5000
 Wire Wire Line
-	1700 1650 1900 1650
-Wire Wire Line
 	1600 1750 1350 1750
 Connection ~ 1200 1750
@@
 P 5300 3050
 F 0 "C48" H 5400 3100 50  0000 L CNN
-F 1 "104" H 5400 2950 50  0000 L CNN
+F 1 "10uF" H 5400 2950 50  0000 L CNN
 F 2 "lc_lib:0805_C" H 5300 3050 50  0001 C CNN
 F 3 "~" H 5300 3050 50  0001 C CNN
@@
 Wire Wire Line
 	3500 5950 3650 5950
-$Comp
-L Device:R_Small JP1
-U 1 1 60390E7A
-P 6050 2550
-F 0 "JP1" H 6109 2596 50  0000 L CNN
-F 1 "0" H 6109 2505 50  0000 L CNN
-F 2 "lc_lib:0805_R" H 6050 2550 50  0001 C CNN
-F 3 "~" H 6050 2550 50  0001 C CNN
-	1    6050 2550
-	0    -1   -1   0
-$EndComp
 Wire Wire Line
 	5950 2550 5300 2550
@@
 	3300 2000 3700 2000
 $Comp
-L Device:CP_Small C63
+L Device:C_Small C63
 U 1 1 60407092
 P 4400 3000
 F 0 "C63" H 4488 3046 50  0000 L CNN
-F 1 "10V 100uF" H 4488 2955 50  0000 L CNN
-F 2 "Capacitor_THT:CP_Radial_D5.0mm_P2.50mm" H 4400 3000 50  0001 C CNN
+F 1 "10uF" H 4488 2955 50  0000 L CNN
+F 2 "lc_lib:0805_C" H 4400 3000 50  0001 C CNN
 F 3 "~" H 4400 3000 50  0001 C CNN
 	1    4400 3000
@@
 	0    1    -1   0
 $EndComp
+Wire Wire Line
+	1200 1650 1900 1650
+$Comp
+L Device:C_Small C68
+U 1 1 6179785C
+P 5400 2000
+F 0 "C68" H 5500 2050 50  0000 L CNN
+F 1 "10uF" H 5500 1900 50  0000 L CNN
+F 2 "lc_lib:0805_C" H 5400 2000 50  0001 C CNN
+F 3 "~" H 5400 2000 50  0001 C CNN
+	1    5400 2000
+	1    0    0    -1
+$EndComp
+Wire Wire Line
+	5400 1900 5400 1650
+Connection ~ 5400 1650
+Wire Wire Line
+	5400 1650 5450 1650
+Wire Wire Line
+	5400 2200 5400 2100
+Wire Wire Line
+	4700 1650 5050 1650
+Wire Wire Line
+	4700 2200 5400 2200
 $EndSCHEMATC

Commit message: routing signals
Parts:
- removed C37: 103, lc_lib:0805_C, symbol Device:C_Small
- FB7: footprint lc_lib:1206_R -> lc_lib:0201_R
Connections:
- net GNDD is gone; now on net GND: FB7.2
- net +5V: no longer R80.2
- net +5VA: now also R80.2
- net GND: no longer FB7.1
- new net GNDA: FB7.1
Other:
- moved on the sheet: D22, R80
Changed lines of the file:
@@
 $Descr A4 11693 8268
 encoding utf-8
-Sheet 5 5
+Sheet 4 5
 Title ""
 Date ""
@@
 Wire Wire Line
 	4700 1900 4700 1650
-Wire Wire Line
-	4700 1650 4550 1650
 Connection ~ 4400 1650
 $Comp
@@
 L Device:R_Small R80
 U 1 1 5E6BDFC2
-P 4550 1300
-F 0 "R80" H 4609 1346 50  0000 L CNN
-F 1 "2.2K" H 4609 1255 50  0000 L CNN
-F 2 "lc_lib:0805_R" H 4550 1300 50  0001 C CNN
-F 3 "~" H 4550 1300 50  0001 C CNN
-	1    4550 1300
+P 4950 1200
+F 0 "R80" H 5009 1246 50  0000 L CNN
+F 1 "2.2K" H 5009 1155 50  0000 L CNN
+F 2 "lc_lib:0805_R" H 4950 1200 50  0001 C CNN
+F 3 "~" H 4950 1200 50  0001 C CNN
+	1    4950 1200
 	1    0    0    -1
 $EndComp
@@
 L MySchLib:LED D22
 U 1 1 5E6BF0FB
-P 4400 1100
-F 0 "D22" H 4393 1316 50  0000 C CNN
-F 1 "Power" H 4393 1225 50  0000 C CNN
-F 2 "lc_lib:0805_LED_S1" H 4400 1100 50  0001 C CNN
-F 3 "~" H 4400 1100 50  0001 C CNN
-	1    4400 1100
-	1    0    0    -1
-$EndComp
-Wire Wire Line
-	4550 1100 4550 1200
-Wire Wire Line
-	4550 1400 4550 1650
-Connection ~ 4550 1650
-Wire Wire Line
-	4550 1650 4400 1650
+P 4800 1000
+F 0 "D22" H 4793 1216 50  0000 C CNN
+F 1 "Power" H 4793 1125 50  0000 C CNN
+F 2 "lc_lib:0805_LED_S1" H 4800 1000 50  0001 C CNN
+F 3 "~" H 4800 1000 50  0001 C CNN
+	1    4800 1000
+	1    0    0    -1
+$EndComp
+Wire Wire Line
+	4950 1000 4950 1100
 $Comp
 L power:GND #PWR0139
 U 1 1 5E6C79FA
-P 4100 1150
-F 0 "#PWR0139" H 4100 900 50  0001 C CNN
-F 1 "GND" H 4105 977 50  0000 C CNN
-F 2 "" H 4100 1150 50  0001 C CNN
-F 3 "" H 4100 1150 50  0001 C CNN
-	1    4100 1150
-	1    0    0    -1
-$EndComp
-Wire Wire Line
-	4100 1150 4100 1100
-Wire Wire Line
-	4100 1100 4250 1100
+P 4500 1050
+F 0 "#PWR0139" H 4500 800 50  0001 C CNN
+F 1 "GND" H 4505 877 50  0000 C CNN
+F 2 "" H 4500 1050 50  0001 C CNN
+F 3 "" H 4500 1050 50  0001 C CNN
+	1    4500 1050
+	1    0    0    -1
+$EndComp
+Wire Wire Line
+	4500 1050 4500 1000
+Wire Wire Line
+	4500 1000 4650 1000
 $Comp
 L Device:Ferrite_Bead_Small FB7
@@
 F 0 "FB7" V 3513 5950 50  0000 C CNN
 F 1 "1K" V 3604 5950 50  0000 C CNN
-F 2 "lc_lib:1206_R" V 3680 5950 50  0001 C CNN
+F 2 "lc_lib:0201_R" V 3680 5950 50  0001 C CNN
 F 3 "~" H 3750 5950 50  0001 C CNN
 	1    3750 5950
@@
 L power:GND #PWR0150
 U 1 1 5E472F1D
-P 4050 6050
-F 0 "#PWR0150" H 4050 5800 50  0001 C CNN
-F 1 "GND" H 4055 5877 50  0000 C CNN
-F 2 "" H 4050 6050 50  0001 C CNN
-F 3 "" H 4050 6050 50  0001 C CNN
-	1    4050 6050
+P 3600 6050
+F 0 "#PWR0150" H 3600 5800 50  0001 C CNN
+F 1 "GND" H 3750 6000 50  0000 C CNN
+F 2 "" H 3600 6050 50  0001 C CNN
+F 3 "" H 3600 6050 50  0001 C CNN
+	1    3600 6050
 	1    0    0    -1
 $EndComp
@@
 	4300 6050 4300 5950
 Wire Wire Line
-	4300 5950 4050 5950
-Wire Wire Line
-	4050 6050 4050 5950
-Connection ~ 4050 5950
-Wire Wire Line
-	4050 5950 3850 5950
+	3600 6050 3600 5950
 $Comp
 L power:GNDD #PWR0152
@@
 	3500 6150 3500 5950
 Wire Wire Line
-	3500 5950 3650 5950
+	3500 5950 3600 5950
 Wire Wire Line
 	5950 2550 5300 2550
@@
 Wire Wire Line
 	1200 3400 850  3400
-$Comp
-L Device:C_Small C37
-U 1 1 6042B935
-P 1350 3450
-F 0 "C37" H 1150 3450 50  0000 L CNN
-F 1 "103" H 1100 3350 50  0000 L CNN
-F 2 "lc_lib:0805_C" H 1350 3450 50  0001 C CNN
-F 3 "~" H 1350 3450 50  0001 C CNN
-	1    1350 3450
-	1    0    0    -1
-$EndComp
 Wire Wire Line
 	1200 3250 1350 3250
@@
 Wire Wire Line
 	1200 3250 1200 3400
-Wire Wire Line
-	1350 3350 1350 3250
 Connection ~ 1350 3250
 Wire Wire Line
@@
 	2000 3250 1600 3250
 Connection ~ 1600 3250
-Wire Wire Line
-	1350 3550 1350 3600
-Wire Wire Line
-	1350 3600 1600 3600
 Wire Wire Line
 	2000 3600 2000 3550
@@
 +5VA
 Wire Wire Line
-	5300 1300 5300 1650
+	5300 1300 5300 1400
 Wire Wire Line
 	3100 2550 5300 2550
@@
 Wire Wire Line
 	4700 2200 5400 2200
+Connection ~ 3600 5950
+Wire Wire Line
+	3600 5950 3650 5950
+Wire Wire Line
+	3850 5950 4300 5950
+Wire Wire Line
+	4400 1650 4700 1650
+Wire Wire Line
+	4950 1300 4950 1400
+Wire Wire Line
+	4950 1400 5300 1400
+Connection ~ 5300 1400
+Wire Wire Line
+	5300 1400 5300 1650
 $EndSCHEMATC

Commit message: almost finished routing MCU2
Parts:
- added R5: 0, lc_lib:0603_R, symbol Device:R_Small
Connections:
- net +5VA: now also R5.2
- net VBL: now also R5.1
Changed lines of the file:
@@
 Wire Wire Line
 	5300 1400 5300 1650
+$Comp
+L Device:R_Small R5
+U 1 1 618FCDB0
+P 6050 2550
+F 0 "R5" V 5854 2550 50  0000 C CNN
+F 1 "0" V 5945 2550 50  0000 C CNN
+F 2 "lc_lib:0603_R" H 6050 2550 50  0001 C CNN
+F 3 "~" H 6050 2550 50  0001 C CNN
+	1    6050 2550
+	0    1    1    0
+$EndComp
 $EndSCHEMATC

Commit message: added EEPROM to MCU
Parts:
- J23: value BIAS -> RF_12V
Connections:
- net BIAS_ON renamed RF_12V_ON
Changed lines of the file:
@@
 P 650 3400
 F 0 "J23" H 568 3617 50  0000 C CNN
-F 1 "BIAS" H 568 3526 50  0000 C CNN
+F 1 "RF_12V" H 568 3526 50  0000 C CNN
 F 2 "Connector_JST:JST_PH_B2B-PH-SM4-TB_1x02-1MP_P2.00mm_Vertical" H 650 3400 50  0001 C CNN
 F 3 "~" H 650 3400 50  0001 C CNN
@@
 	2300 3150 2300 3250
 Text HLabel 2300 3250 3    50   Input ~ 0
-BIAS_ON
+RF_12V_ON
 $Comp
 L Transistor_BJT:DTC144E Q17
