File: RF/OPA2000_RF/RF_input/RF_input.kicad_pcb (KiCad board)
At the start: 2 copper layers, 80 x 100 mm, 145 parts, among them J1 +12V, J2 GND, J3 In, J4 Conn_01x02, J5 Conn_01x02, J6 Conn_01x08, K1 G6K-2, Q1 2N3904, Q2 2N7002K, Q3 2N7002K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

Commit message: MCU2 sch done
Parts:
- removed R24, R47: 22K, lc_lib:0805_R
- removed R48: 47K, lc_lib:0805_R
- added C36: 103, lc_lib:0805_C, F.Cu at (69.2, 104.5)
- added C37: 10uF, lc_lib:0805_C, F.Cu at (69.4, 101.2)
- added C38: 1uF, lc_lib:0805_C, F.Cu at (56.8, 105.8)
- added C39: 104, lc_lib:0805_C, F.Cu at (72.0, 91.5)
- added C40: 102, lc_lib:0805_C, F.Cu at (75.5, 66.2)
- added C41: 102, lc_lib:0805_C, F.Cu at (75.5, 89.8)
- added D17: 8V 1W, lc_lib:SMA(DO-214AC)_S5, F.Cu at (101.5, 67.5)
- added D18: 8V 1W, lc_lib:SMA(DO-214AC)_S5, F.Cu at (101.2, 92.2)
- added D19: 8V 1W, lc_lib:SMA(DO-214AC)_S5, F.Cu at (101.5, 75.8)
- added D20: 8V 1W, lc_lib:SMA(DO-214AC)_S5, F.Cu at (101.2, 84.0)
- added Q10: DTC144E, lc_lib:SOT-23(SOT-23-3), F.Cu at (54.2, 101.0)
- added R56: 100K, lc_lib:0805_R, F.Cu at (58.0, 101.2)
- added R57: 220K, lc_lib:0805_R, F.Cu at (69.2, 98.2)
- added R58: 10K, lc_lib:0805_R, F.Cu at (61.2, 109.2)
- added U5: TLC555xD, lc_lib:SOIC-8_150MIL, F.Cu at (63.2, 100.5)
- C15, C17: value 104 -> 10uF
- J4: value Conn_01x02 -> Imain
- J5: value Conn_01x02 -> Rev
- Q2, Q3: value 2N7002K -> DTC143Z
- Q6: value 2N7002K -> DTC144E
- Q7: value BSS84 -> DTA144E
- R27, R30: value 1 -> 100
- R32, R35, R41: value 1K -> 10K
- R45, R46, R53: value 1K -> 100
- moved R54 29.9 mm to (32.8, 73.8)
- moved Q3 24.7 mm to (80.8, 69.5)
- moved Q2 23.2 mm to (87.2, 64.5), turned to 180 degrees
- moved R52 21.4 mm to (77.2, 59.2), turned to 0 degrees
- moved C34 20.4 mm to (73.0, 59.2), turned to 0 degrees
- moved D10 10.3 mm to (71.0, 108.5)
- moved D11 10.3 mm to (68.8, 108.5)
- moved D12 10.3 mm to (66.6, 108.5)
- moved D13 10.3 mm to (64.4, 108.4)
- moved R13 5.86 mm to (41.8, 37.8), turned to 270 degrees
- moved Q7 5.80 mm to (69.0, 94.8)
- moved TP2 5.27 mm to (98.0, 49.2)
- moved JP1 3.76 mm to (66.2, 50.5)
- moved Q8 3.76 mm to (65.9, 43.2)
- moved Q9 3.76 mm to (65.9, 47.2)
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Connections:
- D10 pad 2: /Protected -> Net-(D10-Pad2)
- D11 pad 2: /Protected -> Net-(D10-Pad2)
- D12 pad 2: /Protected -> Net-(D10-Pad2)
- D13 pad 2: /Protected -> Net-(D10-Pad2)
- Q8 pad 3: Net-(Q8-Pad3) -> +12V
- R1 pad 2: Net-(Q8-Pad3) -> +12V
Routing:
- net +12V: track 0.00 -> 229.0 mm, vias 0 -> 6
- net GND: track 0.00 -> 97.6 mm, vias 0 -> 41
- net /Protected: track 0.00 -> 64.8 mm, vias 0 -> 6
- net VgSense: track 0.00 -> 55.1 mm, vias 0 -> 2
- net Net-(D4-Pad1): track 0.00 -> 46.7 mm
- net Net-(D8-Pad1): track 0.00 -> 44.9 mm, vias 0 -> 4
- net Net-(C5-Pad1): track 0.00 -> 37.8 mm, vias 0 -> 4
- net Net-(D6-Pad1): track 0.00 -> 37.3 mm, vias 0 -> 4
- net REVSense: track 0.00 -> 37.0 mm
- net ImainFault: track 0.00 -> 32.6 mm, vias 0 -> 2
- net BIAS1: track 0.00 -> 32.4 mm
- net PrtctSig: track 0.00 -> 28.5 mm, vias 0 -> 2
- net BIAS2: track 0.00 -> 25.8 mm
- net ImainSense: track 0.00 -> 25.7 mm
- net REVFault: track 0.00 -> 23.7 mm, vias 0 -> 2
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- added copper zone on F.Cu, net GNDPWR
- added copper zone on F.Cu, net Net-(C28-Pad2)
- added copper zone on F.Cu, net Net-(C30-Pad2)
- added copper zone on F.Cu, net Net-(D17-Pad2)
- added copper zone on F.Cu, net Net-(D18-Pad2)
- added copper zone on F.Cu, net Net-(D3-Pad1)

Commit message: almost finished routing MCU2
Parts:
- removed the Q5 at (115.8, 80.0)
- removed R13, R54: 0, lc_lib:0805_R
- added Q11: BLF188XR, MyPCBLib:BLF188XR, F.Cu at (115.8, 80.0)
- D2, D3: value 4148 -> SD103
- R27, R30: value 100 -> 2.2
- moved R20 0.75 mm to (87.8, 57.2)
- turned C13 to 180 degrees
Connections:
- C12 pad 2: GNDPWR -> GND
- C13 pad 1: GNDPWR -> GND
- C14 pad 2: GNDPWR -> GND
- C15 pad 2: GNDPWR -> GND
- C16 pad 2: GNDPWR -> GND
- C17 pad 2: GNDPWR -> GND
- C18 pad 1: GNDPWR -> GND
- C19 pad 2: GNDPWR -> GND
- C32 pad 1: GNDPWR -> GND
- C33 pad 1: GNDPWR -> GND
- D15 pad 2: GNDPWR -> GND
- D16 pad 2: GNDPWR -> GND
- D17 pad 1: GNDPWR -> GND
- D18 pad 1: GNDPWR -> GND
- J3 pad 2: GNDPWR -> GND
- K1 pad 2: GNDPWR -> GND
- K1 pad 3: GNDPWR -> GND
- K1 pad 6: GNDPWR -> GND
- K1 pad 7: GNDPWR -> GND
- R11 pad 1: GNDPWR -> GND
- R12 pad 1: GNDPWR -> GND
- R18 pad 2: GNDPWR -> GND
- R7 pad 1: GNDPWR -> GND
- R8 pad 1: GNDPWR -> GND
- SC1 pad 1: GNDPWR -> GND
- SC2 pad 1: GNDPWR -> GND
- SC3 pad 1: GNDPWR -> GND
- SC4 pad 1: GNDPWR -> GND
- T1 pad 2: GNDPWR -> GND
Routing:
- net PwrOnSig: track 16.0 -> 88.6 mm, vias 2 -> 3
- net BIAS2: track 25.8 -> 43.4 mm
- net G2: track 12.8 -> 30.0 mm
- net G1: track 22.2 -> 38.5 mm
- net +12V: track 229.0 -> 242.1 mm, vias 6 -> 8
- net Net-(R18-Pad1): track 0.00 -> 7.11 mm
- net Net-(R20-Pad2): track 15.7 -> 8.95 mm
- net GND: track 97.6 -> 104.0 mm, vias 41 -> 180
- net GNDPWR: track 6.40 -> 0.00 mm, vias 1 -> 0
- net BIAS1: track 32.4 -> 37.5 mm
- net Net-(R25-Pad2): track 5.47 -> 9.61 mm
- net Net-(D2-Pad1): track 7.56 -> 3.51 mm
- net Net-(C13-Pad2): track 0.00 -> 3.57 mm
- net /Protected: track 64.8 -> 67.4 mm
- net Net-(C10-Pad2): track 10.9 -> 13.4 mm
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- added copper zone on F.Cu, net GND
- added copper zone on In2.Cu, net GND
- added copper zone on F.Cu, net Net-(D2-Pad1)
- added copper zone on F.Cu, net Net-(R18-Pad1)
- removed copper zone on F.Cu, net GNDPWR
Other:
- copper layers 2 -> 4
- board text added: "+12V"
