File: RF/OPA2000_RF/RF_input/RF_input.sch (KiCad schematic (older format))
At the start: 144 parts, among them J1 +12V, J2 GND, J3 In, J4 Conn_01x02, J5 Conn_01x02, J6 Conn_01x08, K1 G6K-2, Q1 2N3904, Q2 2N7002K, Q3 2N7002K, Q4 BLF188XR, Q5 BLF188XR, Q6 2N7002K, Q7 BSS84, Q8 AO3401A, Q9 2N7002, T1 Transformer_4_1, U1 TL431, U2 LM358, U3 LM358, U4 LM324

Commit message: MCU2 sch done
Parts:
- removed Q2, Q3, Q6: 2N7002K, lc_lib:SOT-23(SOT-23-3), symbol Transistor_FET:2N7002K
- removed Q7: BSS84, lc_lib:SOT-23(SOT-23-3), symbol Transistor_FET:BSS84
- removed R24, R47: 22K, lc_lib:0805_R, symbol Device:R_Small
- removed R48: 47K, lc_lib:0805_R, symbol Device:R_Small
- added C36: 103, lc_lib:0805_C, symbol Device:C_Small
- added C37: 10uF, lc_lib:0805_C, symbol Device:C_Small
- added C38: 1uF, lc_lib:0805_C, symbol Device:C_Small
- added C39: 104, lc_lib:0805_C, symbol Device:C_Small
- added C40, C41: 102, lc_lib:0805_C, symbol Device:C_Small
- added D17, D18, D19, D20: 8V 1W, lc_lib:SMA(DO-214AC)_S5, symbol MySchLib:D_Zener
- added Q10, Q6: DTC144E, lc_lib:SOT-23(SOT-23-3), symbol Transistor_BJT:DTC144E
- added Q2, Q3: DTC143Z, lc_lib:SOT-23(SOT-23-3), symbol Transistor_BJT:DTC143Z
- added Q7: DTA144E, lc_lib:SOT-23(SOT-23-3), symbol Transistor_BJT:DTA144E
- added R56: 100K, lc_lib:0805_R, symbol Device:R_Small
- added R57: 220K, lc_lib:0805_R, symbol Device:R_Small
- added R58: 10K, lc_lib:0805_R, symbol Device:R_Small
- added U5: TLC555xD, lc_lib:SOIC-8_150MIL, symbol Timer:TLC555xD
- C15, C17: value 104 -> 10uF
- D2, D3: value 4148 -> SD103
- J4: value Conn_01x02 -> Imain
- J5: value Conn_01x02 -> Rev
- Q4, Q5: symbol MySchLib:BLF188XR -> RF_input-rescue:BLF188XR-MySchLib
- R27, R30: value 1 -> 100
- R32, R35, R41: value 1K -> 10K
- R45, R46, R53: value 1K -> 100
Connections:
- wire segments 431 -> 476
Other:
- moved on the sheet: C22, C24, D10, D11, D12, D13, J4, J5, R36, R38, R43, R44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

Commit message: almost finished routing MCU2
Parts:
- removed R13, R54: 0, lc_lib:0805_R, symbol Device:R_Small
- added Q11: BLF188XR, MyPCBLib:BLF188XR, symbol RF_input-rescue:BLF188XR-MySchLib
- D5, D7, D9: symbol MySchLib:LED -> RF_input-rescue:LED-MySchLib
- R27, R30: value 100 -> 2.2
Connections:
- net GNDPWR is gone; now on net GND: C12.2, C13.1, C14.2, C15.2, C16.2, C17.2, C18.1, C19.2, C32.1, C33.1, D15.2 (K), D16.2 (K), D17.1 (A), D18.1 (A), J3.2 (Ext), K1.2, K1.3, K1.6, K1.7, R11.1, R12.1, R18.2, R7.1, R8.1, SC1.1 (Pin_1), SC2.1 (Pin_1), SC3.1 (Pin_1), SC4.1 (Pin_1), T1.2 (AB)
- net G1: now also Q11.3 (G)
- net G2: now also Q11.4 (G)
Changed lines of the file:
@@
 	1    0    0    -1
 $EndComp
-$Comp
-L power:GND #PWR06
-U 1 1 5DE8EEF6
-P 2350 2750
-F 0 "#PWR06" H 2350 2500 50  0001 C CNN
-F 1 "GND" H 2355 2577 50  0000 C CNN
-F 2 "" H 2350 2750 50  0001 C CNN
-F 3 "" H 2350 2750 50  0001 C CNN
-	1    2350 2750
-	1    0    0    -1
-$EndComp
-$Comp
-L power:GND #PWR016
-U 1 1 5DE9895A
-P 3050 2350
-F 0 "#PWR016" H 3050 2100 50  0001 C CNN
-F 1 "GND" H 3055 2177 50  0000 C CNN
-F 2 "" H 3050 2350 50  0001 C CNN
-F 3 "" H 3050 2350 50  0001 C CNN
-	1    3050 2350
-	1    0    0    -1
-$EndComp
 Wire Wire Line
 	3050 2350 3050 2050
 Wire Wire Line
 	3050 1250 3050 1350
-$Comp
-L Device:C_Small C3
-U 1 1 5DE9E430
-P 2850 1350
-F 0 "C3" V 2621 1350 50  0000 C CNN
-F 1 "104" V 2712 1350 50  0000 C CNN
-F 2 "lc_lib:0805_C" H 2850 1350 50  0001 C CNN
-F 3 "~" H 2850 1350 50  0001 C CNN
-	1    2850 1350
-	0    1    1    0
-$EndComp
 Wire Wire Line
 	2950 1350 3050 1350
@@
 	1    0    0    -1
 $EndComp
-$Comp
-L Device:R_Small R13
-U 1 1 5DE96617
-P 3550 7150
-F 0 "R13" H 3609 7196 50  0000 L CNN
-F 1 "0" H 3609 7105 50  0000 L CNN
-F 2 "lc_lib:0805_R" H 3609 7059 50  0001 L CNN
-F 3 "~" H 3550 7150 50  0001 C CNN
-	1    3550 7150
-	0    -1   -1   0
-$EndComp
 Wire Wire Line
 	3300 7250 3300 7150
 Wire Wire Line
-	3300 7150 3450 7150
-Wire Wire Line
-	3650 7150 3850 7150
-Wire Wire Line
 	3850 7150 3850 7250
 Wire Wire Line
@@
 	1    0    0    -1
 $EndComp
-$Comp
-L power:GND #PWR014
-U 1 1 60A69076
-P 2950 3850
-F 0 "#PWR014" H 2950 3600 50  0001 C CNN
-F 1 "GND" H 2955 3677 50  0000 C CNN
-F 2 "" H 2950 3850 50  0001 C CNN
-F 3 "" H 2950 3850 50  0001 C CNN
-	1    2950 3850
-	1    0    0    -1
-$EndComp
 Wire Wire Line
 	2950 3850 2950 3700
@@
 Wire Wire Line
 	2950 3000 2950 3100
-$Comp
-L power:GND #PWR017
-U 1 1 60ABCAFB
-P 3250 3050
-F 0 "#PWR017" H 3250 2800 50  0001 C CNN
-F 1 "GND" H 3255 2877 50  0000 C CNN
-F 2 "" H 3250 3050 50  0001 C CNN
-F 3 "" H 3250 3050 50  0001 C CNN
-	1    3250 3050
-	1    0    0    -1
-$EndComp
 Wire Wire Line
 	3200 3000 3250 3000
@@
 Wire Wire Line
 	1700 3400 1700 3500
-$Comp
-L power:GND #PWR05
-U 1 1 60B01EDF
-P 1700 3850
-F 0 "#PWR05" H 1700 3600 50  0001 C CNN
-F 1 "GND" H 1705 3677 50  0000 C CNN
-F 2 "" H 1700 3850 50  0001 C CNN
-F 3 "" H 1700 3850 50  0001 C CNN
-	1    1700 3850
-	1    0    0    -1
-$EndComp
 Wire Wire Line
 	1700 3700 1700 3850
-$Comp
-L power:GND #PWR09
-U 1 1 60B1F2C3
-P 2050 3800
-F 0 "#PWR09" H 2050 3550 50  0001 C CNN
-F 1 "GND" H 2055 3627 50  0000 C CNN
-F 2 "" H 2050 3800 50  0001 C CNN
-F 3 "" H 2050 3800 50  0001 C CNN
-	1    2050 3800
-	1    0    0    -1
-$EndComp
 Wire Wire Line
 	2050 3800 2050 3700
@@
 P 5500 6550
 F 0 "R30" H 5559 6596 50  0000 L CNN
-F 1 "100" H 5559 6505 50  0000 L CNN
+F 1 "2.2" H 5559 6505 50  0000 L CNN
 F 2 "lc_lib:1206_R" H 5559 6459 50  0001 L CNN
 F 3 "~" H 5500 6550 50  0001 C CNN
@@
 P 5500 4800
 F 0 "R27" H 5559 4846 50  0000 L CNN
-F 1 "100" H 5559 4755 50  0000 L CNN
+F 1 "2.2" H 5559 4755 50  0000 L CNN
 F 2 "MyPCBLib:L_Axial_0.4_SMD" H 5559 4709 50  0001 L CNN
 F 3 "~" H 5500 4800 50  0001 C CNN
@@
 ImainFault
 $Comp
-L MySchLib:LED D5
+L RF_input-rescue:LED-MySchLib D5
 U 1 1 6096AD85
 P 7050 1600
@@
 $EndComp
 $Comp
-L MySchLib:LED D7
+L RF_input-rescue:LED-MySchLib D7
 U 1 1 60B6878A
 P 8100 1600
@@
 $EndComp
 $Comp
-L MySchLib:LED D9
+L RF_input-rescue:LED-MySchLib D9
 U 1 1 60E2F9D7
 P 9000 1650
@@
 BIAS2
 Wire Wire Line
-	10350 2400 9650 2400
-Wire Wire Line
-	9650 2400 9650 3500
-Wire Wire Line
-	9650 3500 5900 3500
-Wire Wire Line
-	5900 3500 5900 4450
-Wire Wire Line
-	5900 4450 5500 4450
-Wire Wire Line
-	5500 4450 5500 4550
-Connection ~ 5500 4550
-Wire Wire Line
 	6050 4550 6450 4550
 $Comp
@@
 $EndComp
 $Comp
-L Device:R_Small R54
-U 1 1 6240E21D
-P 4400 7150
-F 0 "R54" H 4459 7196 50  0000 L CNN
-F 1 "0" H 4459 7105 50  0000 L CNN
-F 2 "lc_lib:0805_R" H 4459 7059 50  0001 L CNN
-F 3 "~" H 4400 7150 50  0001 C CNN
-	1    4400 7150
-	0    -1   -1   0
-$EndComp
-$Comp
-L power:GND #PWR0104
-U 1 1 6240E5C6
-P 4200 7250
-F 0 "#PWR0104" H 4200 7000 50  0001 C CNN
-F 1 "GND" H 4205 7077 50  0000 C CNN
-F 2 "" H 4200 7250 50  0001 C CNN
-F 3 "" H 4200 7250 50  0001 C CNN
-	1    4200 7250
-	1    0    0    -1
-$EndComp
-Wire Wire Line
-	4200 7250 4200 7150
-Wire Wire Line
-	4200 7150 4300 7150
-$Comp
-L power:GNDPWR #PWR0105
-U 1 1 6243F411
-P 4600 7250
-F 0 "#PWR0105" H 4600 7050 50  0001 C CNN
-F 1 "GNDPWR" H 4604 7096 50  0000 C CNN
-F 2 "" H 4600 7200 50  0001 C CNN
-F 3 "" H 4600 7200 50  0001 C CNN
-	1    4600 7250
-	1    0    0    -1
-$EndComp
-Wire Wire Line
-	4600 7250 4600 7150
-Wire Wire Line
-	4600 7150 4500 7150
-$Comp
 L power:+12V #PWR0106
 U 1 1 6114AD86
@@
 	5700 5150 6100 5150
 Wire Wire Line
-	6100 5150 6100 5300
+	6100 5150 6100 5200
 Connection ~ 6100 5150
 Connection ~ 5750 5650
@@
 	5900 5750 5900 5650
 Connection ~ 5900 5650
+Entry Wire Line
+	4700 1500 4800 1600
+$Comp
+L power:GNDPWR #PWR0104
+U 1 1 618A916F
+P 2350 2750
+F 0 "#PWR0104" H 2350 2550 50  0001 C CNN
+F 1 "GNDPWR" H 2354 2596 50  0000 C CNN
+F 2 "" H 2350 2700 50  0001 C CNN
+F 3 "" H 2350 2700 50  0001 C CNN
+	1    2350 2750
+	1    0    0    -1
+$EndComp
+$Comp
+L Device:C_Small C3
+U 1 1 5DE9E430
+P 2850 1350
+F 0 "C3" V 2621 1350 50  0000 C CNN
+F 1 "104" V 2712 1350 50  0000 C CNN
+F 2 "lc_lib:0805_C" H 2850 1350 50  0001 C CNN
+F 3 "~" H 2850 1350 50  0001 C CNN
+	1    2850 1350
+	0    1    1    0
+$EndComp
+$Comp
+L power:GND #PWR016
+U 1 1 5DE9895A
+P 3050 2350
+F 0 "#PWR016" H 3050 2100 50  0001 C CNN
+F 1 "GND" H 3055 2177 50  0000 C CNN
+F 2 "" H 3050 2350 50  0001 C CNN
+F 3 "" H 3050 2350 50  0001 C CNN
+	1    3050 2350
+	1    0    0    -1
+$EndComp
+$Comp
+L power:GND #PWR017
+U 1 1 60ABCAFB
+P 3250 3050
+F 0 "#PWR017" H 3250 2800 50  0001 C CNN
+F 1 "GND" H 3255 2877 50  0000 C CNN
+F 2 "" H 3250 3050 50  0001 C CNN
+F 3 "" H 3250 3050 50  0001 C CNN
+	1    3250 3050
+	1    0    0    -1
+$EndComp
+$Comp
+L power:GND #PWR014
+U 1 1 60A69076
+P 2950 3850
+F 0 "#PWR014" H 2950 3600 50  0001 C CNN
+F 1 "GND" H 2955 3677 50  0000 C CNN
+F 2 "" H 2950 3850 50  0001 C CNN
+F 3 "" H 2950 3850 50  0001 C CNN
+	1    2950 3850
+	1    0    0    -1
+$EndComp
+$Comp
+L power:GND #PWR09
+U 1 1 60B1F2C3
+P 2050 3800
+F 0 "#PWR09" H 2050 3550 50  0001 C CNN
+F 1 "GND" H 2055 3627 50  0000 C CNN
+F 2 "" H 2050 3800 50  0001 C CNN
+F 3 "" H 2050 3800 50  0001 C CNN
+	1    2050 3800
+	1    0    0    -1
+$EndComp
+$Comp
+L power:GND #PWR05
+U 1 1 60B01EDF
+P 1700 3850
+F 0 "#PWR05" H 1700 3600 50  0001 C CNN
+F 1 "GND" H 1705 3677 50  0000 C CNN
+F 2 "" H 1700 3850 50  0001 C CNN
+F 3 "" H 1700 3850 50  0001 C CNN
+	1    1700 3850
+	1    0    0    -1
+$EndComp
+Wire Wire Line
+	3300 7150 3850 7150
+Wire Wire Line
+	9550 2400 9550 3600
+Wire Wire Line
+	9550 3600 6300 3600
+Wire Wire Line
+	6300 3600 6300 3750
+Wire Wire Line
+	6300 3750 5500 3750
+Wire Wire Line
+	5500 3750 5500 4550
+Wire Wire Line
+	9550 2400 10350 2400
+Connection ~ 5500 4550
+$Comp
+L RF_input-rescue:BLF188XR-MySchLib Q11
+U 1 1 61B51440
+P 6600 5650
+F 0 "Q11" H 6700 5400 50  0000 L CNN
+F 1 "BLF188XR" H 6650 5300 50  0000 L CNN
+F 2 "MyPCBLib:BLF188XR" H 6600 5780 50  0001 C CNN
+F 3 "" H 6600 5780 50  0001 C CNN
+	1    6600 5650
+	1    0    0    -1
+$EndComp
+Wire Wire Line
+	6300 5500 6300 5200
+Wire Wire Line
+	6300 5200 6100 5200
+Connection ~ 6100 5200
+Wire Wire Line
+	6100 5200 6100 5300
+Wire Wire Line
+	6300 5800 6300 5950
+Wire Wire Line
+	6300 5950 6200 5950
+Wire Wire Line
+	6200 5950 6200 6050
+Wire Wire Line
+	6200 6050 6100 6050
+Connection ~ 6100 6050
 $EndSCHEMATC
